File: E-MATCH/REV A/E-MATCH.sch (KiCad schematic (older format))
At the start: 2 parts

Commit message: REV B Pogo
Parts:
- P1: renamed from P?; footprint (none) -> MOD:4 PAD E-MATCH
- P2: renamed from P?; footprint (none) -> MOD:200MIL_ST
Changed lines of the file:
@@
 LIBS:contrib
 LIBS:valves
+LIBS:E-MATCH-cache
 EELAYER 25 0
 EELAYER END
@@
 $EndDescr
 $Comp
-L CONN_01X04 P?
+L CONN_01X04 P2
 U 1 1 5A5580EB
 P 6250 3850
-F 0 "P?" H 6250 4100 50  0000 C CNN
+F 0 "P2" H 6250 4100 50  0000 C CNN
 F 1 "E-MATCH" H 6500 3850 50  0000 C CNN
-F 2 "" H 6250 3850 50  0000 C CNN
+F 2 "MOD:200MIL_ST" H 6250 3850 50  0001 C CNN
 F 3 "" H 6250 3850 50  0000 C CNN
 	1    6250 3850
@@
 $EndComp
 $Comp
-L CONN_01X02 P?
+L CONN_01X02 P1
 U 1 1 5A55813C
 P 5750 3750
-F 0 "P?" H 5750 3900 50  0000 C CNN
+F 0 "P1" H 5750 3900 50  0000 C CNN
 F 1 "SCREW TERMINAL" H 6150 3750 50  0000 C CNN
-F 2 "" H 5750 3750 50  0000 C CNN
+F 2 "MOD:4 PAD E-MATCH" H 5750 3750 50  0001 C CNN
 F 3 "" H 5750 3750 50  0000 C CNN
 	1    5750 3750
