File: MAIN BOARD/REV B/MAIN.kicad_pcb (KiCad board)
At the start: 2 copper layers, 54.6 x 29.2 mm, 179 parts, among them J1 502570-0893, P1 SERVO 1, P2 SERVO 2, P3 SERVO 3, P4 E-MATCH, P5 SERVO 4, P6 SERVO 5, P7 PVC, P8 LIPO, P9 USB_OTG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

Commit message: REV B Pogo
Connections:
- U4 pad 8: SERVO_EN -> 8V_FUSE
- U4 pad 9: (no net) -> GND
Routing:
- net 8V_FUSE: track 22.3 -> 27.3 mm
- net GND: track 53.1 -> 54.1 mm, vias 6 -> 8
- net (no net): track 0.98 -> 0.00 mm, vias 2 -> 0
