File: MAIN BOARD/REV B/MAIN.sch (KiCad schematic (older format))
At the start: 62 parts, among them J1 502570-0893, P1 SERVO 1, P2 SERVO 2, P3 SERVO 3, P4 E-MATCH, P5 SERVO 4, P6 SERVO 5, P7 PVC, P8 LIPO, P9 USB_OTG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

Commit message: REV B Pogo
Connections:
- net SERVO_EN is gone; now on net 8V_FUSE: U4.8 (EN)
Other:
- moved on the sheet: C14, C15, C18, C19, C20, C21, D2, D4, F2, P9, R3, R4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
