File: STATION/REV A/MAIN.kicad_pcb (KiCad board)
At the start: 2 copper layers, 22.4 x 29.2 mm, 84 parts, among them P9 USB_OTG, SW1 Push_SW, U1 AX5043, U2 AP1117, U5 ATMEGA32U2, Y1 16MHz, Y2 8MHz

Commit message: REV B Pogo
Other:
- board text added: "MICRO USB"
- board text added: "MOUNTING HOLES"
- board text added: "U.FL CONN."
- board text added: "ZIP TIE TO HOLD DOWN COAX CABLE"
Changed lines of the file:
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@@
 (kicad_pcb (version 4) (host pcbnew 4.0.5+dfsg1-4)
   (general
-    (links 0)
+    (links 135)
     (no_connects 0)
-    (area 94.387998 82.449999 116.940001 111.860001)
+    (area 74.282299 81.1113 117.8607 112.9077)
     (thickness 1.6)
-    (drawings 13)
+    (drawings 27)
     (tracks 216)
     (zones 0)
@@
       (xy 3.878332 1.547088) (xy 3.839633 1.582875) (xy 3.877733 1.582957) (xy 3.900277 1.581843)) (layer B.SilkS) (width 0.01))
   )
+  (gr_text "ZIP TIE TO HOLD\nDOWN COAX CABLE" (at 86.106 71.374) (layer Eco2.User)
+    (effects (font (size 1.5 1.5) (thickness 0.3)))
+  )
+  (gr_line (start 114.3 95.25) (end 97.028 73.914) (layer Eco2.User) (width 0.2))
+  (gr_line (start 128.27 77.724) (end 114.3 109.22) (layer Eco2.User) (width 0.2))
+  (gr_text "MOUNTING HOLES" (at 139.192 77.978) (layer Eco2.User)
+    (effects (font (size 1.5 1.5) (thickness 0.3)))
+  )
+  (gr_line (start 114.3 85.09) (end 128.27 77.724) (layer Eco2.User) (width 0.2))
+  (gr_text "MICRO USB" (at 75.946 79.756) (layer Eco2.User)
+    (effects (font (size 1.5 1.5) (thickness 0.3)))
+  )
+  (gr_line (start 95.758 86.106) (end 82.55 79.756) (layer Eco2.User) (width 0.2))
+  (gr_text "U.FL CONN." (at 137.414 83.566) (layer Eco2.User)
+    (effects (font (size 1.5 1.5) (thickness 0.3)))
+  )
+  (gr_line (start 115.824 90.424) (end 130.81 83.566) (layer Eco2.User) (width 0.2))
+  (dimension 2.54 (width 0.3) (layer Eco1.User)
+    (gr_text "0.1000 in" (at 87.804 109.22 270) (layer Eco1.User)
+      (effects (font (size 1.5 1.5) (thickness 0.3)))
+    )
+    (feature1 (pts (xy 114.3 110.49) (xy 86.454 110.49)))
+    (feature2 (pts (xy 114.3 107.95) (xy 86.454 107.95)))
+    (crossbar (pts (xy 89.154 107.95) (xy 89.154 110.49)))
+    (arrow1a (pts (xy 89.154 110.49) (xy 88.567579 109.363496)))
+    (arrow1b (pts (xy 89.154 110.49) (xy 89.740421 109.363496)))
+    (arrow2a (pts (xy 89.154 107.95) (xy 88.567579 109.076504)))
+    (arrow2b (pts (xy 89.154 107.95) (xy 89.740421 109.076504)))
+  )
+  (dimension 2.54 (width 0.3) (layer Eco1.User)
+    (gr_text "0.1000 in" (at 126.064 110.49 270) (layer Eco1.User)
+      (effects (font (size 1.5 1.5) (thickness 0.3)))
+    )
+    (feature1 (pts (xy 114.3 111.76) (xy 127.414 111.76)))
+    (feature2 (pts (xy 114.3 109.22) (xy 127.414 109.22)))
+    (crossbar (pts (xy 124.714 109.22) (xy 124.714 111.76)))
+    (arrow1a (pts (xy 124.714 111.76) (xy 124.127579 110.633496)))
+    (arrow1b (pts (xy 124.714 111.76) (xy 125.300421 110.633496)))
+    (arrow2a (pts (xy 124.714 109.22) (xy 124.127579 110.346504)))
+    (arrow2b (pts (xy 124.714 109.22) (xy 125.300421 110.346504)))
+  )
+  (dimension 2.54 (width 0.3) (layer Eco1.User)
+    (gr_text "0.1000 in" (at 115.57 116.158) (layer Eco1.User)
+      (effects (font (size 1.5 1.5) (thickness 0.3)))
+    )
+    (feature1 (pts (xy 116.84 109.22) (xy 116.84 117.508)))
+    (feature2 (pts (xy 114.3 109.22) (xy 114.3 117.508)))
+    (crossbar (pts (xy 114.3 114.808) (xy 116.84 114.808)))
+    (arrow1a (pts (xy 116.84 114.808) (xy 115.713496 115.394421)))
+    (arrow1b (pts (xy 116.84 114.808) (xy 115.713496 114.221579)))
+    (arrow2a (pts (xy 114.3 114.808) (xy 115.426504 115.394421)))
+    (arrow2b (pts (xy 114.3 114.808) (xy 115.426504 114.221579)))
+  )
+  (dimension 29.21 (width 0.3) (layer Eco1.User)
+    (gr_text "1.1500 in" (at 123.016 97.155 270) (layer Eco1.User)
+      (effects (font (size 1.5 1.5) (thickness 0.3)))
+    )
+    (feature1 (pts (xy 116.84 111.76) (xy 124.366 111.76)))
+    (feature2 (pts (xy 116.84 82.55) (xy 124.366 82.55)))
+    (crossbar (pts (xy 121.666 82.55) (xy 121.666 111.76)))
+    (arrow1a (pts (xy 121.666 111.76) (xy 121.079579 110.633496)))
+    (arrow1b (pts (xy 121.666 111.76) (xy 122.252421 110.633496)))
+    (arrow2a (pts (xy 121.666 82.55) (xy 121.079579 83.676504)))
+    (arrow2b (pts (xy 121.666 82.55) (xy 122.252421 83.676504)))
+  )
+  (dimension 22.352 (width 0.3) (layer Eco1.User)
+    (gr_text "0.8800 in" (at 105.664 77.39) (layer Eco1.User)
+      (effects (font (size 1.5 1.5) (thickness 0.3)))
+    )
+    (feature1 (pts (xy 94.488 82.55) (xy 94.488 76.04)))
+    (feature2 (pts (xy 116.84 82.55) (xy 116.84 76.04)))
+    (crossbar (pts (xy 116.84 78.74) (xy 94.488 78.74)))
+    (arrow1a (pts (xy 94.488 78.74) (xy 95.614504 78.153579)))
+    (arrow1b (pts (xy 94.488 78.74) (xy 95.614504 79.326421)))
+    (arrow2a (pts (xy 116.84 78.74) (xy 115.713496 78.153579)))
+    (arrow2b (pts (xy 116.84 78.74) (xy 115.713496 79.326421)))
+  )
   (gr_text "CDM REV A\n12-4-17" (at 97.917 84.074 180) (layer B.Cu)
